File: RXProg.kicad_pcb (KiCad board)
At the start: 4 copper layers, 18.8 x 36.6 mm, 25 parts, among them J1 Conn_01x14, J2 Conn_01x14, J3 Pin, J4 Pin, J5 USB_B_Micro, J6 SWD, U1 STM32G474CETx, U2 SN74ALVC164245DL, U3 TXU0104RUTR, U4 MIC5317-3.3xM5, U5 FXMA108

Commit message: Finish routing (again)
Parts:
- C11: moved to B.Cu
- C7: moved to F.Cu
- U2: value SN74ALVC164245DL -> SN74ALVC164245DGG; footprint Package_SO:SSOP-48_7.5x15.9mm_P0.635mm -> Package_SO:TSSOP-48_6.1x12.5mm_P0.5mm
- moved C11 9.25 mm to (131.3, 102.5), turned to 90 degrees
- moved J3 2.20 mm to (130.8, 116.4)
- moved J4 2.20 mm to (130.8, 118.6)
- moved C7 1.50 mm to (131.3, 94.1), turned to 180 degrees
- moved C9 0.97 mm to (127.8, 97.4), turned to 180 degrees
- moved U2 0.95 mm to (126.2, 106.0)
- moved C10 0.82 mm to (123.6, 101.2)
- moved C1 0.81 mm to (131.1, 102.5)
- moved C8 0.66 mm to (127.2, 92.4), turned to 90 degrees
- moved C4 0.50 mm to (121.6, 111.1)
- moved C2 0.20 mm to (130.2, 102.7)
- moved C3 0.10 mm to (129.9, 112.1)
Routing:
- net /VBAT: track 29.6 -> 43.5 mm, vias 8 -> 5
- net GND: track 46.5 -> 36.3 mm, vias 19 -> 28
- net ~{CS1}: track 28.3 -> 20.2 mm
- net +3V3: track 20.9 -> 27.5 mm, vias 6 -> 7
- net A8: track 27.5 -> 21.9 mm
- net ~{ADDR_OE}: track 23.2 -> 17.7 mm
- net ~{NRST}: track 16.6 -> 11.4 mm, vias 2 -> 0
- net Net-(U1-PB10): track 11.4 -> 16.0 mm
- net D5: track 13.1 -> 17.2 mm
- net A9: track 17.5 -> 21.2 mm
- net Net-(J6-SWCLK): track 24.2 -> 20.6 mm
- net Net-(U1-PB5): track 3.67 -> 0.47 mm
- net Net-(U1-PB12): track 13.2 -> 16.3 mm, vias 3 -> 2
- net ~{CS3}: track 21.2 -> 24.1 mm
- net Net-(U1-PB4): track 3.83 -> 1.05 mm
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- added copper zone on In2.Cu, net +3V3
- added copper zone on B.Cu, net GND
- added copper zone on F.Cu, net GND
- added copper zone on In4.Cu, net GND
- added copper zone on In2.Cu, net /VBAT
- removed copper zone on In2.Cu, net GND
- removed copper zone on B.Cu, net /VBAT
Other:
- copper layers 4 -> 6
- board text added: "CS2"
- board text added: "CS3"
- board text added: "Max Pastushkov 2026"
- board text added: "Yamaha RX USB Interface"
